File: src/PCB/KiCAD/huzzah_ct.kicad_pcb (KiCad board)
At the start: 2 copper layers, 6 parts, among them CON1 BARREL_JACK, U1 MCP3008, U2 DS18B20, U3 Adafruit_HUZZAH, U4 LM317T

Commit message: pcb routing
Parts:
- added C1: 0.1uF, Capacitors_ThroughHole:C_Radial_D5_L11_P2, F.Cu at (64.8, 57.1)
- added C2: 10uF, Capacitors_ThroughHole:C_Radial_D5_L11_P2, F.Cu at (82.5, 64.8)
- added R2: 150, Resistors_ThroughHole:Resistor_Horizontal_RM7mm, F.Cu at (97.8, 59.7)
- added R3: 150, Resistors_ThroughHole:Resistor_Horizontal_RM7mm, F.Cu at (86.4, 59.7)
- added R4: 150, Resistors_ThroughHole:Resistor_Horizontal_RM7mm, F.Cu at (90.2, 63.5)
- moved U4 79.1 mm to (73.7, 59.7), turned to 90 degrees
- moved CON1 53.1 mm to (48.3, 57.1)
- moved R1 37.0 mm to (67.3, 67.3)
Connections:
- CON1 pad 1: Net-(CON1-Pad1) -> Net-(C1-Pad1)
- CON1 pad 2: Net-(CON1-Pad2) -> GNDREF
- R1 pad 1: Net-(R1-Pad1) -> Net-(C2-Pad1)
- R1 pad 2: Net-(R1-Pad2) -> GNDREF
- U4 pad 1: Net-(U4-Pad1) -> Net-(C2-Pad1)
- U4 pad 3: Net-(U4-Pad3) -> Net-(C1-Pad1)
Routing:
- net GNDREF: track 0.00 -> 58.3 mm
- net Net-(C2-Pad1): track 0.00 -> 26.5 mm
- net Net-(C1-Pad1): track 0.00 -> 19.3 mm
- net Net-(R3-Pad2): track 0.00 -> 5.08 mm
- net Net-(R2-Pad2): track 0.00 -> 3.81 mm
- net Net-(R2-Pad1): track 0.00 -> 3.81 mm
